File: pcb/lintilla.kicad_pcb (KiCad board)
At the start: 2 copper layers, 157.4 x 111.6 mm, 71 parts

Commit message: Change to supermini, add power jack, mirror design
Parts:
- removed the ? at (68.1, 34.8)
- removed the ? at (173.3, 111.7)
- removed the ? at (149.4, 45.0)
- removed the ? at (81.5, 106.2)
- removed ARC1: , arc_guide
- removed G*** (x4): LOGO, Graphics:Lintilla
- removed G*** (x4): LOGO, Graphics:Allitnil
- removed PAD1, PAD2, PAD3, PAD4, PAD5, PAD6: , SMDPad
- removed V1, V2, V3, V4, V5: VIA-0.6mm, VIA-0.6mm
- added ?: , MountingHole_2.2mm_M2_Pad_Via, F.Cu at (315.7, 41.3)
- added ?: , MountingHole_2.2mm_M2_Pad_Via, F.Cu at (164.5, 127.6)
- added ?: , MountingHole_2.2mm_M2_Pad_Via, F.Cu at (308.6, 113.6)
- added ?: , MountingHole_2.2mm_M2_Pad_Via, F.Cu at (73.5, 114.2)
- added ?: , MountingHole_2.2mm_M2_Pad_Via, F.Cu at (235.6, 58.5)
- added ?: , MountingHole_2.2mm_M2_Pad_Via, F.Cu at (217.6, 127.0)
- added ?: , MountingHole_2.2mm_M2_Pad_Via, F.Cu at (146.5, 59.1)
- added ?: , MountingHole_2.2mm_M2_Pad_Via, F.Cu at (66.4, 41.9)
- added JST1: , ceoloide:battery_connector_jst_ph_2, F.Cu at (170.4, 86.8)
- added JST1: , ceoloide:battery_connector_jst_ph_2, B.Cu at (211.7, 86.4)
- added MCU2: , ceoloide:mcu_supermini_nrf52840, F.Cu at (221.3, 63.8)
- added S22: , PG1350, F.Cu at (341.0, 103.4)
- added S23: , PG1350, F.Cu at (343.4, 85.5)
- added S24: , PG1350, F.Cu at (321.6, 109.2)
- added S25: , PG1350, F.Cu at (323.9, 91.4)
- added S26: , PG1350, F.Cu at (326.3, 73.5)
- added S27: , PG1350, F.Cu at (328.2, 46.8)
- added S28: , PG1350, F.Cu at (304.8, 94.7)
- added S29: , PG1350, F.Cu at (305.6, 76.7)
- added S30: , PG1350, F.Cu at (306.4, 58.7)
- added S31: , PG1350, F.Cu at (286.5, 84.7)
- added S32: , PG1350, F.Cu at (285.6, 66.7)
- added S33: , PG1350, F.Cu at (284.6, 48.7)
- added S34: , PG1350, F.Cu at (268.7, 94.7)
- added S35: , PG1350, F.Cu at (267.1, 76.8)
- added S36: , PG1350, F.Cu at (265.5, 58.8)
- added S37: , PG1350, F.Cu at (250.5, 99.4)
- added S38: , PG1350, F.Cu at (248.9, 81.4)
- added S39: , PG1350, F.Cu at (247.4, 63.5)
- added S40: , PG1350, F.Cu at (250.3, 118.5)
- added S41: , PG1350, F.Cu at (232.0, 127.9)
- added S42: , PG1350, F.Cu at (216.8, 141.8)
- added SW22: , ComboDiode, F.Cu at (341.5, 99.7)
- added SW23: , ComboDiode, F.Cu at (343.8, 81.8)
- added SW24: , ComboDiode, F.Cu at (322.1, 105.5)
- added SW25: , ComboDiode, F.Cu at (324.4, 87.6)
- added SW26: , ComboDiode, F.Cu at (326.8, 69.8)
- added SW27: , ComboDiode, F.Cu at (328.1, 43.0)
- added SW28: , ComboDiode, F.Cu at (305.0, 90.9)
- added SW29: , ComboDiode, F.Cu at (305.8, 73.0)
- added SW30: , ComboDiode, F.Cu at (306.6, 55.0)
- added SW31: , ComboDiode, F.Cu at (286.4, 80.9)
- added SW32: , ComboDiode, F.Cu at (285.4, 62.9)
- added SW33: , ComboDiode, F.Cu at (284.4, 45.0)
- added SW34: , ComboDiode, F.Cu at (268.3, 91.0)
- added SW35: , ComboDiode, F.Cu at (266.8, 73.0)
- added SW36: , ComboDiode, F.Cu at (265.2, 55.1)
- added SW37: , ComboDiode, F.Cu at (250.2, 95.6)
- added SW38: , ComboDiode, F.Cu at (248.6, 77.7)
- added SW39: , ComboDiode, F.Cu at (247.0, 59.8)
- added SW40: , ComboDiode, F.Cu at (249.0, 115.0)
- added SW41: , ComboDiode, F.Cu at (229.9, 124.9)
- added SW42: , ComboDiode, F.Cu at (213.9, 139.4)
- MCU1: footprint xiao-ble -> ceoloide:mcu_supermini_nrf52840
- moved B2 151.5 mm to (267.8, 50.1), turned to 5 degrees
- moved T2 115.1 mm to (249.6, 54.7), turned to 5 degrees
- moved SW21 19.1 mm to (168.2, 140.0), turned to 130 degrees
- moved S21 19.0 mm to (165.3, 142.4), turned to 130 degrees
- moved SW20 17.3 mm to (152.2, 125.5), turned to 145 degrees
- moved S20 17.2 mm to (150.1, 128.5), turned to 145 degrees
- moved S19 15.5 mm to (131.8, 119.1), turned to 160 degrees
- moved SW19 15.4 mm to (133.1, 115.6), turned to 160 degrees
- moved S16 14.6 mm to (131.6, 100.0), turned to 175 degrees
- moved SW16 14.4 mm to (131.9, 96.2), turned to 175 degrees
- moved S17 14.0 mm to (133.2, 82.0), turned to 175 degrees
- moved SW17 13.9 mm to (133.5, 78.3), turned to 175 degrees
- moved MCU1 13.8 mm to (160.8, 64.4), turned to -5 degrees
- moved S18 13.6 mm to (134.7, 64.1), turned to 175 degrees
- moved SW18 13.5 mm to (135.1, 60.4), turned to 175 degrees
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Connections:
- MCU1 pad 1: (no net) -> P1
- MCU1 pad 10: P9 -> P7
- MCU1 pad 11: P10 -> P8
- MCU1 pad 12: (no net) -> P9
- MCU1 pad 13: GND -> P10
- MCU1 pad 14: (no net) -> P16
- MCU1 pad 15: GND -> P14
- MCU1 pad 16: P2 -> P15
- MCU1 pad 17: P3 -> P18
- MCU1 pad 18: P4 -> P19
- MCU1 pad 19: P5 -> P20
- MCU1 pad 2: P1 -> P0
- MCU1 pad 20: P6 -> P21
- MCU1 pad 21: P1 -> VCC
- MCU1 pad 22: P10 -> RST
- MCU1 pad 23: P9 -> GND
- MCU1 pad 24: P8 -> RAW
- MCU1 pad 3: P2 -> GND
- MCU1 pad 4: P3 -> GND
- MCU1 pad 5: P4 -> P2
- MCU1 pad 6: P5 -> P3
- MCU1 pad 7: P6 -> P4
- MCU1 pad 8: P7 -> P5
- MCU1 pad 9: P8 -> P6
- T2 pad 1: (no net) -> BAT+
- T2 pad 3: BAT+ -> RAW
Routing:
- net GND: track 233.3 -> 0.00 mm
- net P1: track 231.0 -> 0.00 mm
- net P8: track 218.9 -> 0.00 mm
- net P4: track 209.2 -> 0.00 mm
- net P9: track 206.4 -> 0.00 mm
- net P2: track 193.4 -> 0.00 mm
- net P3: track 178.2 -> 0.00 mm
- net P7: track 171.8 -> 0.00 mm
- net P5: track 171.5 -> 0.00 mm
- net P10: track 159.5 -> 0.00 mm
- net P6: track 148.6 -> 0.00 mm
- net RST: track 80.6 -> 0.00 mm
- net RAW: track 77.0 -> 0.00 mm
- net BAT+: track 54.9 -> 0.00 mm
- net outer_home: track 17.2 -> 0.00 mm
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- removed copper zone on B.Cu, net GND
- removed copper zone on F.Cu, net GND
Other:
- board size 157.4 x 111.6 mm -> 328.4 x 120.4 mm
- rule pad_to_mask_clearance: 0 -> 0.05
- board text added: "https://github.com/nathankrish/lintilla"
- board text added: "v1.1"
- board text removed: "Allitnil"
- board text removed: "BATTERY 5 x 20 x 30 mm"
- board text removed: "Licensed under CERN-OHL-P v2"
- board text removed: "XIAO BLE FACE DOWN"
- board text removed: "https://github.com/ctranstrum/lintilla"
- board text removed: "solder all components same side"
- board text removed: "v1.0"
